File: hardware/blinkybadge.sch (KiCad schematic (older format))
At the start: 21 parts, among them IC101 ATMEGA8U2, P101 USB_OTG, P102 CONN_02X03, Q101 Q_PMOS_GDS, SW101 SPST, U101 ATECC508A, Y101 16MHz

Commit message: More layout
Connections:
- net VBAT: now also SW101.2; no longer SW101.1
- net VBAT_SW: now also SW101.1; no longer SW101.2
- net USBR_P: now reaches IC101.29 (D+), R101.1
- net USBR_N: now reaches IC101.30 (D-), R102.1
- net USB_DN renamed USB_N
- net USB_DP renamed USB_P
Other:
- moved on the sheet: R101, R102
Changed lines of the file:
@@
 F 3 "" H 3850 2000 50  0000 C CNN
 	1    3850 2000
-	1    0    0    -1
+	-1   0    0    -1
 $EndComp
 $Comp
@@
 STAT
 Text Label 1950 2100 2    60   ~ 0
-USB_DN
+USB_N
 Text Label 1950 2200 2    60   ~ 0
-USB_DP
+USB_P
 $Comp
 L R R101
 U 1 1 577C8F67
-P 4150 4750
-F 0 "R101" V 4230 4750 50  0000 C CNN
-F 1 "22" V 4150 4750 50  0000 C CNN
-F 2 "Resistors_SMD:R_0603" V 4080 4750 50  0001 C CNN
-F 3 "" H 4150 4750 50  0000 C CNN
-	1    4150 4750
+P 3800 4750
+F 0 "R101" V 3880 4750 50  0000 C CNN
+F 1 "22" V 3800 4750 50  0000 C CNN
+F 2 "Resistors_SMD:R_0603" V 3730 4750 50  0001 C CNN
+F 3 "" H 3800 4750 50  0000 C CNN
+	1    3800 4750
 	0    1    1    0
 $EndComp
@@
 L R R102
 U 1 1 577C90FD
-P 4150 4850
-F 0 "R102" V 4230 4850 50  0000 C CNN
-F 1 "22" V 4150 4850 50  0000 C CNN
-F 2 "Resistors_SMD:R_0603" V 4080 4850 50  0001 C CNN
-F 3 "" H 4150 4850 50  0000 C CNN
-	1    4150 4850
-	0    1    1    0
-$EndComp
-Text Label 3500 4750 0    60   ~ 0
-USB_DP
-Text Label 3500 4850 0    60   ~ 0
-USB_DN
+P 3800 4850
+F 0 "R102" V 3880 4850 50  0000 C CNN
+F 1 "22" V 3800 4850 50  0000 C CNN
+F 2 "Resistors_SMD:R_0603" V 3730 4850 50  0001 C CNN
+F 3 "" H 3800 4850 50  0000 C CNN
+	1    3800 4850
+	0    1    1    0
+$EndComp
+Text Label 3150 4750 0    60   ~ 0
+USB_P
+Text Label 3150 4850 0    60   ~ 0
+USB_N
 $Comp
 L VCC #PWR05
@@
 	1600 2400 1600 2600
 Wire Wire Line
-	1500 2000 2300 2000
+	1500 2000 1950 2000
+Wire Wire Line
+	1950 2000 2300 2000
 Wire Wire Line
 	3350 2000 3000 2000
@@
 	5100 1600 5100 1700
 Wire Wire Line
-	1950 1600 5500 1600
+	1950 1600 4400 1600
+Wire Wire Line
+	4400 1600 5100 1600
+Wire Wire Line
+	5100 1600 5500 1600
 Wire Wire Line
 	1950 1600 1950 2000
@@
 Connection ~ 5100 1600
 Wire Wire Line
-	5300 2000 5700 2000
-Wire Wire Line
-	5700 1700 5700 2950
+	5300 2000 5500 2000
+Wire Wire Line
+	5500 2000 5700 2000
+Wire Wire Line
+	5700 1700 5700 2000
+Wire Wire Line
+	5700 2000 5700 2850
+Wire Wire Line
+	5700 2850 5700 2950
 Connection ~ 5500 2000
 Wire Wire Line
@@
 	1500 2200 1950 2200
 Wire Wire Line
-	4300 4750 4600 4750
-Wire Wire Line
-	4300 4850 4600 4850
-Wire Wire Line
-	4000 4750 3500 4750
-Wire Wire Line
-	4000 4850 3500 4850
+	3950 4750 4600 4750
+Wire Wire Line
+	3950 4850 4600 4850
+Wire Wire Line
+	3650 4750 3150 4750
+Wire Wire Line
+	3650 4850 3150 4850
 Connection ~ 5700 2000
 Wire Wire Line
@@
 	4400 4550 4400 5000
 Wire Wire Line
-	4400 5300 4400 5400
+	4400 5300 4400 5350
+Wire Wire Line
+	4400 5350 4400 5400
 Wire Wire Line
 	4600 4950 4600 5350
@@
 Connection ~ 4400 5350
 Wire Wire Line
-	4000 4050 4400 4050
+	4000 4050 4200 4050
+Wire Wire Line
+	4200 4050 4400 4050
 Wire Wire Line
 	4400 3850 4600 3850
@@
 	4400 3750 4400 3850
 Wire Wire Line
-	4000 3750 4400 3750
+	4000 3750 4200 3750
+Wire Wire Line
+	4200 3750 4400 3750
 Wire Wire Line
 	4600 3950 4400 3950
@@
 	3700 3750 3550 3750
 Wire Wire Line
-	3550 3750 3550 4200
+	3550 3750 3550 4050
+Wire Wire Line
+	3550 4050 3550 4200
 Connection ~ 3550 4050
 Wire Wire Line
@@
 	8000 3650 8000 3550
 Wire Wire Line
-	4150 2850 5700 2850
-Wire Wire Line
-	4500 2850 4500 4650
+	4150 2850 4500 2850
+Wire Wire Line
+	4500 2850 5700 2850
+Wire Wire Line
+	4500 2850 4500 3750
+Wire Wire Line
+	4500 3750 4500 4650
 Wire Wire Line
 	4500 3750 4600 3750
@@
 	8950 4150 9100 4150
 Wire Wire Line
-	6800 5050 7300 5050
+	6800 5050 7250 5050
+Wire Wire Line
+	7250 5050 7300 5050
 Wire Wire Line
 	6800 5150 6900 5150
@@
 Wire Wire Line
 	8000 3850 8200 3850
+Text Label 4000 4750 0    60   ~ 0
+USBR_P
+Text Label 4000 4850 0    60   ~ 0
+USBR_N
 $EndSCHEMATC
