File: hardware/LEDs.sch (KiCad schematic (older format))
At the start: 12 parts

Commit message: Moar LEDs
Parts:
- added C? (x2): 1uF, symbol C
- added D? (x2): WS2812B, WS2812B, symbol WS2812B
Connections:
- net GND: now also C?.2, C?.2, D?.3 (VSS), D?.3 (VSS)
- net VCC: now also C?.1, C?.1, D?.1 (VDD), D?.1 (VDD)
- new net: D?.2 (DOUT), D?.4 (DIN)
- new net DOUT: D?.2 (DOUT)
Other:
- moved on the sheet: C?, D?

Commit message: Add annotations
Parts:
- gave numbers to parts that had none: 16
Changed lines of the file:
@@
 DIN
 $Comp
-L WS2812B D?
+L WS2812B D301
 U 1 1 577DCBE1
 P 3350 3300
-F 0 "D?" H 3010 3580 50  0000 L CNN
+F 0 "D301" H 3010 3580 50  0000 L CNN
 F 1 "WS2812B" H 3200 3300 50  0000 L CNN
 F 2 "WS2812B" H 3200 3300 50  0001 L CNN
@@
 	2600 3150 2900 3150
 $Comp
-L C C?
+L C C301
 U 1 1 577DCCC3
 P 3350 2900
-F 0 "C?" H 3375 3000 50  0000 L CNN
+F 0 "C301" H 3375 3000 50  0000 L CNN
 F 1 "1uF" H 3375 2800 50  0000 L CNN
 F 2 "" H 3388 2750 50  0000 C CNN
@@
 	3900 2900 3500 2900
 $Comp
-L WS2812B D?
+L WS2812B D303
 U 1 1 577DCD4A
 P 4800 3300
-F 0 "D?" H 4460 3580 50  0000 L CNN
+F 0 "D303" H 4460 3580 50  0000 L CNN
 F 1 "WS2812B" H 4650 3300 50  0000 L CNN
 F 2 "WS2812B" H 4650 3300 50  0001 L CNN
@@
 	4050 3150 4350 3150
 $Comp
-L C C?
+L C C303
 U 1 1 577DCD51
 P 4800 2900
-F 0 "C?" H 4825 3000 50  0000 L CNN
+F 0 "C303" H 4825 3000 50  0000 L CNN
 F 1 "1uF" H 4825 2800 50  0000 L CNN
 F 2 "" H 4838 2750 50  0000 C CNN
@@
 	4050 3450 4050 3150
 $Comp
-L WS2812B D?
+L WS2812B D305
 U 1 1 577DCDD7
 P 6250 3300
-F 0 "D?" H 5910 3580 50  0000 L CNN
+F 0 "D305" H 5910 3580 50  0000 L CNN
 F 1 "WS2812B" H 6100 3300 50  0000 L CNN
 F 2 "WS2812B" H 6100 3300 50  0001 L CNN
@@
 	5500 3150 5800 3150
 $Comp
-L C C?
+L C C305
 U 1 1 577DCDDE
 P 6250 2900
-F 0 "C?" H 6275 3000 50  0000 L CNN
+F 0 "C305" H 6275 3000 50  0000 L CNN
 F 1 "1uF" H 6275 2800 50  0000 L CNN
 F 2 "" H 6288 2750 50  0000 C CNN
@@
 	6800 2900 6400 2900
 $Comp
-L WS2812B D?
+L WS2812B D307
 U 1 1 577DCE44
 P 7700 3300
-F 0 "D?" H 7360 3580 50  0000 L CNN
+F 0 "D307" H 7360 3580 50  0000 L CNN
 F 1 "WS2812B" H 7550 3300 50  0000 L CNN
 F 2 "WS2812B" H 7550 3300 50  0001 L CNN
@@
 	6950 3150 7250 3150
 $Comp
-L C C?
+L C C307
 U 1 1 577DCE4B
 P 7700 2900
-F 0 "C?" H 7725 3000 50  0000 L CNN
+F 0 "C307" H 7725 3000 50  0000 L CNN
 F 1 "1uF" H 7725 2800 50  0000 L CNN
 F 2 "" H 7738 2750 50  0000 C CNN
@@
 	8250 2900 7850 2900
 $Comp
-L WS2812B D?
+L WS2812B D302
 U 1 1 577DCEC5
 P 3350 4900
-F 0 "D?" H 3010 5180 50  0000 L CNN
+F 0 "D302" H 3010 5180 50  0000 L CNN
 F 1 "WS2812B" H 3200 4900 50  0000 L CNN
 F 2 "WS2812B" H 3200 4900 50  0001 L CNN
@@
 	2600 4750 2900 4750
 $Comp
-L C C?
+L C C302
 U 1 1 577DCECC
 P 3350 4500
-F 0 "C?" H 3375 4600 50  0000 L CNN
+F 0 "C302" H 3375 4600 50  0000 L CNN
 F 1 "1uF" H 3375 4400 50  0000 L CNN
 F 2 "" H 3388 4350 50  0000 C CNN
@@
 	3900 4500 3500 4500
 $Comp
-L WS2812B D?
+L WS2812B D304
 U 1 1 577DCF4A
 P 4800 4900
-F 0 "D?" H 4460 5180 50  0000 L CNN
+F 0 "D304" H 4460 5180 50  0000 L CNN
 F 1 "WS2812B" H 4650 4900 50  0000 L CNN
 F 2 "WS2812B" H 4650 4900 50  0001 L CNN
@@
 	4050 4750 4350 4750
 $Comp
-L C C?
+L C C304
 U 1 1 577DCF51
 P 4800 4500
-F 0 "C?" H 4825 4600 50  0000 L CNN
+F 0 "C304" H 4825 4600 50  0000 L CNN
 F 1 "1uF" H 4825 4400 50  0000 L CNN
 F 2 "" H 4838 4350 50  0000 C CNN
@@
 Connection ~ 4250 3450
 $Comp
-L GND #PWR?
+L GND #PWR302
 U 1 1 577DD399
 P 7150 3900
-F 0 "#PWR?" H 7150 3650 50  0001 C CNN
+F 0 "#PWR302" H 7150 3650 50  0001 C CNN
 F 1 "GND" H 7150 3750 50  0000 C CNN
 F 2 "" H 7150 3900 50  0000 C CNN
@@
 $EndComp
 $Comp
-L VCC #PWR?
+L VCC #PWR301
 U 1 1 577DD41D
 P 6800 2550
-F 0 "#PWR?" H 6800 2400 50  0001 C CNN
+F 0 "#PWR301" H 6800 2400 50  0001 C CNN
 F 1 "VCC" H 6800 2700 50  0000 C CNN
 F 2 "" H 6800 2550 50  0000 C CNN
@@
 	3900 2700 8550 2700
 $Comp
-L WS2812B D?
+L WS2812B D306
 U 1 1 577DEFF8
 P 6250 4900
-F 0 "D?" H 5910 5180 50  0000 L CNN
+F 0 "D306" H 5910 5180 50  0000 L CNN
 F 1 "WS2812B" H 6100 4900 50  0000 L CNN
 F 2 "WS2812B" H 6100 4900 50  0001 L CNN
@@
 	5500 4750 5800 4750
 $Comp
-L C C?
+L C C306
 U 1 1 577DEFFF
 P 6250 4500
-F 0 "C?" H 6275 4600 50  0000 L CNN
+F 0 "C306" H 6275 4600 50  0000 L CNN
 F 1 "1uF" H 6275 4400 50  0000 L CNN
 F 2 "" H 6288 4350 50  0000 C CNN
@@
 	6800 4500 6400 4500
 $Comp
-L WS2812B D?
+L WS2812B D308
 U 1 1 577DF00B
 P 7700 4900
-F 0 "D?" H 7360 5180 50  0000 L CNN
+F 0 "D308" H 7360 5180 50  0000 L CNN
 F 1 "WS2812B" H 7550 4900 50  0000 L CNN
 F 2 "WS2812B" H 7550 4900 50  0001 L CNN
@@
 	6950 4750 7250 4750
 $Comp
-L C C?
+L C C308
 U 1 1 577DF012
 P 7700 4500
-F 0 "C?" H 7725 4600 50  0000 L CNN
+F 0 "C308" H 7725 4600 50  0000 L CNN
 F 1 "1uF" H 7725 4400 50  0000 L CNN
 F 2 "" H 7738 4350 50  0000 C CNN

Commit message: Update footprints
Parts:
- C301, C302, C303, C304, C305, C306, C307, C308: footprint (none) -> Capacitors_SMD:C_0603
Changed lines of the file:
@@
 F 0 "C301" H 3375 3000 50  0000 L CNN
 F 1 "1uF" H 3375 2800 50  0000 L CNN
-F 2 "" H 3388 2750 50  0000 C CNN
+F 2 "Capacitors_SMD:C_0603" H 3388 2750 50  0001 C CNN
 F 3 "" H 3350 2900 50  0000 C CNN
 	1    3350 2900
@@
 F 0 "C303" H 4825 3000 50  0000 L CNN
 F 1 "1uF" H 4825 2800 50  0000 L CNN
-F 2 "" H 4838 2750 50  0000 C CNN
+F 2 "Capacitors_SMD:C_0603" H 4838 2750 50  0001 C CNN
 F 3 "" H 4800 2900 50  0000 C CNN
 	1    4800 2900
@@
 F 0 "C305" H 6275 3000 50  0000 L CNN
 F 1 "1uF" H 6275 2800 50  0000 L CNN
-F 2 "" H 6288 2750 50  0000 C CNN
+F 2 "Capacitors_SMD:C_0603" H 6288 2750 50  0001 C CNN
 F 3 "" H 6250 2900 50  0000 C CNN
 	1    6250 2900
@@
 F 0 "C307" H 7725 3000 50  0000 L CNN
 F 1 "1uF" H 7725 2800 50  0000 L CNN
-F 2 "" H 7738 2750 50  0000 C CNN
+F 2 "Capacitors_SMD:C_0603" H 7738 2750 50  0001 C CNN
 F 3 "" H 7700 2900 50  0000 C CNN
 	1    7700 2900
@@
 F 0 "C302" H 3375 4600 50  0000 L CNN
 F 1 "1uF" H 3375 4400 50  0000 L CNN
-F 2 "" H 3388 4350 50  0000 C CNN
+F 2 "Capacitors_SMD:C_0603" H 3388 4350 50  0001 C CNN
 F 3 "" H 3350 4500 50  0000 C CNN
 	1    3350 4500
@@
 F 0 "C304" H 4825 4600 50  0000 L CNN
 F 1 "1uF" H 4825 4400 50  0000 L CNN
-F 2 "" H 4838 4350 50  0000 C CNN
+F 2 "Capacitors_SMD:C_0603" H 4838 4350 50  0001 C CNN
 F 3 "" H 4800 4500 50  0000 C CNN
 	1    4800 4500
@@
 Connection ~ 4250 3450
 $Comp
-L GND #PWR302
+L GND #PWR014
 U 1 1 577DD399
 P 7150 3900
-F 0 "#PWR302" H 7150 3650 50  0001 C CNN
+F 0 "#PWR014" H 7150 3650 50  0001 C CNN
 F 1 "GND" H 7150 3750 50  0000 C CNN
 F 2 "" H 7150 3900 50  0000 C CNN
@@
 $EndComp
 $Comp
-L VCC #PWR301
+L VCC #PWR015
 U 1 1 577DD41D
 P 6800 2550
-F 0 "#PWR301" H 6800 2400 50  0001 C CNN
+F 0 "#PWR015" H 6800 2400 50  0001 C CNN
 F 1 "VCC" H 6800 2700 50  0000 C CNN
 F 2 "" H 6800 2550 50  0000 C CNN
@@
 F 0 "C306" H 6275 4600 50  0000 L CNN
 F 1 "1uF" H 6275 4400 50  0000 L CNN
-F 2 "" H 6288 4350 50  0000 C CNN
+F 2 "Capacitors_SMD:C_0603" H 6288 4350 50  0001 C CNN
 F 3 "" H 6250 4500 50  0000 C CNN
 	1    6250 4500
@@
 F 0 "C308" H 7725 4600 50  0000 L CNN
 F 1 "1uF" H 7725 4400 50  0000 L CNN
-F 2 "" H 7738 4350 50  0000 C CNN
+F 2 "Capacitors_SMD:C_0603" H 7738 4350 50  0001 C CNN
 F 3 "" H 7700 4500 50  0000 C CNN
 	1    7700 4500

Commit message: Update some footprint assignments
Parts:
- D301, D302, D303, D304, D305, D306, D307, D308: footprint WS2812B -> (none)
Changed lines of the file:
@@
 F 0 "D301" H 3010 3580 50  0000 L CNN
 F 1 "WS2812B" H 3200 3300 50  0000 L CNN
-F 2 "WS2812B" H 3200 3300 50  0001 L CNN
+F 2 "" H 3200 3300 50  0001 L CNN
 F 3 "" H 3100 3250 60  0000 C CNN
 	1    3350 3300
@@
 F 0 "D303" H 4460 3580 50  0000 L CNN
 F 1 "WS2812B" H 4650 3300 50  0000 L CNN
-F 2 "WS2812B" H 4650 3300 50  0001 L CNN
+F 2 "" H 4650 3300 50  0001 L CNN
 F 3 "" H 4550 3250 60  0000 C CNN
 	1    4800 3300
@@
 F 0 "D305" H 5910 3580 50  0000 L CNN
 F 1 "WS2812B" H 6100 3300 50  0000 L CNN
-F 2 "WS2812B" H 6100 3300 50  0001 L CNN
+F 2 "" H 6100 3300 50  0001 L CNN
 F 3 "" H 6000 3250 60  0000 C CNN
 	1    6250 3300
@@
 F 0 "D307" H 7360 3580 50  0000 L CNN
 F 1 "WS2812B" H 7550 3300 50  0000 L CNN
-F 2 "WS2812B" H 7550 3300 50  0001 L CNN
+F 2 "" H 7550 3300 50  0001 L CNN
 F 3 "" H 7450 3250 60  0000 C CNN
 	1    7700 3300
@@
 F 0 "D302" H 3010 5180 50  0000 L CNN
 F 1 "WS2812B" H 3200 4900 50  0000 L CNN
-F 2 "WS2812B" H 3200 4900 50  0001 L CNN
+F 2 "" H 3200 4900 50  0001 L CNN
 F 3 "" H 3100 4850 60  0000 C CNN
 	1    3350 4900
@@
 F 0 "D304" H 4460 5180 50  0000 L CNN
 F 1 "WS2812B" H 4650 4900 50  0000 L CNN
-F 2 "WS2812B" H 4650 4900 50  0001 L CNN
+F 2 "" H 4650 4900 50  0001 L CNN
 F 3 "" H 4550 4850 60  0000 C CNN
 	1    4800 4900
@@
 F 0 "D306" H 5910 5180 50  0000 L CNN
 F 1 "WS2812B" H 6100 4900 50  0000 L CNN
-F 2 "WS2812B" H 6100 4900 50  0001 L CNN
+F 2 "" H 6100 4900 50  0001 L CNN
 F 3 "" H 6000 4850 60  0000 C CNN
 	1    6250 4900
@@
 F 0 "D308" H 7360 5180 50  0000 L CNN
 F 1 "WS2812B" H 7550 4900 50  0000 L CNN
-F 2 "WS2812B" H 7550 4900 50  0001 L CNN
+F 2 "" H 7550 4900 50  0001 L CNN
 F 3 "" H 7450 4850 60  0000 C CNN
 	1    7700 4900

Commit message: Begin layout work
Parts:
- D301, D302, D303, D304, D305, D306, D307, D308: footprint (none) -> LEDs:LED_WS2812B-PLCC4
Changed lines of the file:
@@
 F 0 "D301" H 3010 3580 50  0000 L CNN
 F 1 "WS2812B" H 3200 3300 50  0000 L CNN
-F 2 "" H 3200 3300 50  0001 L CNN
+F 2 "LEDs:LED_WS2812B-PLCC4" H 3200 3300 50  0001 L CNN
 F 3 "" H 3100 3250 60  0000 C CNN
 	1    3350 3300
@@
 F 0 "D303" H 4460 3580 50  0000 L CNN
 F 1 "WS2812B" H 4650 3300 50  0000 L CNN
-F 2 "" H 4650 3300 50  0001 L CNN
+F 2 "LEDs:LED_WS2812B-PLCC4" H 4650 3300 50  0001 L CNN
 F 3 "" H 4550 3250 60  0000 C CNN
 	1    4800 3300
@@
 F 0 "D305" H 5910 3580 50  0000 L CNN
 F 1 "WS2812B" H 6100 3300 50  0000 L CNN
-F 2 "" H 6100 3300 50  0001 L CNN
+F 2 "LEDs:LED_WS2812B-PLCC4" H 6100 3300 50  0001 L CNN
 F 3 "" H 6000 3250 60  0000 C CNN
 	1    6250 3300
@@
 F 0 "D307" H 7360 3580 50  0000 L CNN
 F 1 "WS2812B" H 7550 3300 50  0000 L CNN
-F 2 "" H 7550 3300 50  0001 L CNN
+F 2 "LEDs:LED_WS2812B-PLCC4" H 7550 3300 50  0001 L CNN
 F 3 "" H 7450 3250 60  0000 C CNN
 	1    7700 3300
@@
 F 0 "D302" H 3010 5180 50  0000 L CNN
 F 1 "WS2812B" H 3200 4900 50  0000 L CNN
-F 2 "" H 3200 4900 50  0001 L CNN
+F 2 "LEDs:LED_WS2812B-PLCC4" H 3200 4900 50  0001 L CNN
 F 3 "" H 3100 4850 60  0000 C CNN
 	1    3350 4900
@@
 F 0 "D304" H 4460 5180 50  0000 L CNN
 F 1 "WS2812B" H 4650 4900 50  0000 L CNN
-F 2 "" H 4650 4900 50  0001 L CNN
+F 2 "LEDs:LED_WS2812B-PLCC4" H 4650 4900 50  0001 L CNN
 F 3 "" H 4550 4850 60  0000 C CNN
 	1    4800 4900
@@
 F 0 "D306" H 5910 5180 50  0000 L CNN
 F 1 "WS2812B" H 6100 4900 50  0000 L CNN
-F 2 "" H 6100 4900 50  0001 L CNN
+F 2 "LEDs:LED_WS2812B-PLCC4" H 6100 4900 50  0001 L CNN
 F 3 "" H 6000 4850 60  0000 C CNN
 	1    6250 4900
@@
 F 0 "D308" H 7360 5180 50  0000 L CNN
 F 1 "WS2812B" H 7550 4900 50  0000 L CNN
-F 2 "" H 7550 4900 50  0001 L CNN
+F 2 "LEDs:LED_WS2812B-PLCC4" H 7550 4900 50  0001 L CNN
 F 3 "" H 7450 4850 60  0000 C CNN
 	1    7700 4900

Commit message: Layout complete
Parts:
- renumbered C303 to C302, C305 to C303, C307 to C304, C302 to C305, C304 to C306, C306 to C307, D303 to D302, D305 to D303, D307 to D304, D302 to D305, D304 to D306, D306 to D307
Connections:
- net at D306.2 (DOUT): now also D307.4 (DIN)
Changed lines of the file:
@@
 	3900 2900 3500 2900
 $Comp
-L WS2812B D303
+L WS2812B D302
 U 1 1 577DCD4A
 P 4800 3300
-F 0 "D303" H 4460 3580 50  0000 L CNN
+F 0 "D302" H 4460 3580 50  0000 L CNN
 F 1 "WS2812B" H 4650 3300 50  0000 L CNN
 F 2 "LEDs:LED_WS2812B-PLCC4" H 4650 3300 50  0001 L CNN
@@
 	4050 3150 4350 3150
 $Comp
-L C C303
+L C C302
 U 1 1 577DCD51
 P 4800 2900
-F 0 "C303" H 4825 3000 50  0000 L CNN
+F 0 "C302" H 4825 3000 50  0000 L CNN
 F 1 "1uF" H 4825 2800 50  0000 L CNN
 F 2 "Capacitors_SMD:C_0603" H 4838 2750 50  0001 C CNN
@@
 	4050 3450 4050 3150
 $Comp
-L WS2812B D305
+L WS2812B D303
 U 1 1 577DCDD7
 P 6250 3300
-F 0 "D305" H 5910 3580 50  0000 L CNN
+F 0 "D303" H 5910 3580 50  0000 L CNN
 F 1 "WS2812B" H 6100 3300 50  0000 L CNN
 F 2 "LEDs:LED_WS2812B-PLCC4" H 6100 3300 50  0001 L CNN
@@
 	5500 3150 5800 3150
 $Comp
-L C C305
+L C C303
 U 1 1 577DCDDE
 P 6250 2900
-F 0 "C305" H 6275 3000 50  0000 L CNN
+F 0 "C303" H 6275 3000 50  0000 L CNN
 F 1 "1uF" H 6275 2800 50  0000 L CNN
 F 2 "Capacitors_SMD:C_0603" H 6288 2750 50  0001 C CNN
@@
 	6800 2900 6400 2900
 $Comp
-L WS2812B D307
+L WS2812B D304
 U 1 1 577DCE44
 P 7700 3300
-F 0 "D307" H 7360 3580 50  0000 L CNN
+F 0 "D304" H 7360 3580 50  0000 L CNN
 F 1 "WS2812B" H 7550 3300 50  0000 L CNN
 F 2 "LEDs:LED_WS2812B-PLCC4" H 7550 3300 50  0001 L CNN
@@
 	6950 3150 7250 3150
 $Comp
-L C C307
+L C C304
 U 1 1 577DCE4B
 P 7700 2900
-F 0 "C307" H 7725 3000 50  0000 L CNN
+F 0 "C304" H 7725 3000 50  0000 L CNN
 F 1 "1uF" H 7725 2800 50  0000 L CNN
 F 2 "Capacitors_SMD:C_0603" H 7738 2750 50  0001 C CNN
@@
 	8250 2900 7850 2900
 $Comp
-L WS2812B D302
+L WS2812B D305
 U 1 1 577DCEC5
 P 3350 4900
-F 0 "D302" H 3010 5180 50  0000 L CNN
+F 0 "D305" H 3010 5180 50  0000 L CNN
 F 1 "WS2812B" H 3200 4900 50  0000 L CNN
 F 2 "LEDs:LED_WS2812B-PLCC4" H 3200 4900 50  0001 L CNN
@@
 	2600 4750 2900 4750
 $Comp
-L C C302
+L C C305
 U 1 1 577DCECC
 P 3350 4500
-F 0 "C302" H 3375 4600 50  0000 L CNN
+F 0 "C305" H 3375 4600 50  0000 L CNN
 F 1 "1uF" H 3375 4400 50  0000 L CNN
 F 2 "Capacitors_SMD:C_0603" H 3388 4350 50  0001 C CNN
@@
 	3900 4500 3500 4500
 $Comp
-L WS2812B D304
+L WS2812B D306
 U 1 1 577DCF4A
 P 4800 4900
-F 0 "D304" H 4460 5180 50  0000 L CNN
+F 0 "D306" H 4460 5180 50  0000 L CNN
 F 1 "WS2812B" H 4650 4900 50  0000 L CNN
 F 2 "LEDs:LED_WS2812B-PLCC4" H 4650 4900 50  0001 L CNN
@@
 	4050 4750 4350 4750
 $Comp
-L C C304
+L C C306
 U 1 1 577DCF51
 P 4800 4500
-F 0 "C304" H 4825 4600 50  0000 L CNN
+F 0 "C306" H 4825 4600 50  0000 L CNN
 F 1 "1uF" H 4825 4400 50  0000 L CNN
 F 2 "Capacitors_SMD:C_0603" H 4838 4350 50  0001 C CNN
@@
 Connection ~ 4250 3450
 $Comp
-L GND #PWR014
+L GND #PWR015
 U 1 1 577DD399
 P 7150 3900
-F 0 "#PWR014" H 7150 3650 50  0001 C CNN
+F 0 "#PWR015" H 7150 3650 50  0001 C CNN
 F 1 "GND" H 7150 3750 50  0000 C CNN
 F 2 "" H 7150 3900 50  0000 C CNN
@@
 $EndComp
 $Comp
-L VCC #PWR015
+L VCC #PWR016
 U 1 1 577DD41D
 P 6800 2550
-F 0 "#PWR015" H 6800 2400 50  0001 C CNN
+F 0 "#PWR016" H 6800 2400 50  0001 C CNN
 F 1 "VCC" H 6800 2700 50  0000 C CNN
 F 2 "" H 6800 2550 50  0000 C CNN
@@
 	3900 2700 8550 2700
 $Comp
-L WS2812B D306
+L WS2812B D307
 U 1 1 577DEFF8
 P 6250 4900
-F 0 "D306" H 5910 5180 50  0000 L CNN
+F 0 "D307" H 5910 5180 50  0000 L CNN
 F 1 "WS2812B" H 6100 4900 50  0000 L CNN
 F 2 "LEDs:LED_WS2812B-PLCC4" H 6100 4900 50  0001 L CNN
@@
 	5500 4750 5800 4750
 $Comp
-L C C306
+L C C307
 U 1 1 577DEFFF
 P 6250 4500
-F 0 "C306" H 6275 4600 50  0000 L CNN
+F 0 "C307" H 6275 4600 50  0000 L CNN
 F 1 "1uF" H 6275 4400 50  0000 L CNN
 F 2 "Capacitors_SMD:C_0603" H 6288 4350 50  0001 C CNN
@@
 Wire Wire Line
 	8150 5050 8550 5050
+Wire Wire Line
+	5500 4750 5500 5050
+Wire Wire Line
+	5500 5050 5250 5050
 $EndSCHEMATC
