File: hardware/LEDs.sch (KiCad schematic (older format))
At the start: 16 parts

Commit message: Fix PMOS pinout
Parts:
- D301, D302, D303, D304, D305, D306, D307, D308: footprint LEDs:LED_WS2812B-PLCC4 -> lib:LED_WS2812B-PLCC4
Changed lines of the file:
@@
 F 0 "D301" H 3010 3580 50  0000 L CNN
 F 1 "WS2812B" H 3200 3300 50  0000 L CNN
-F 2 "LEDs:LED_WS2812B-PLCC4" H 3200 3300 50  0001 L CNN
+F 2 "lib:LED_WS2812B-PLCC4" H 3200 3300 50  0001 L CNN
 F 3 "" H 3100 3250 60  0000 C CNN
 	1    3350 3300
@@
 F 0 "D302" H 4460 3580 50  0000 L CNN
 F 1 "WS2812B" H 4650 3300 50  0000 L CNN
-F 2 "LEDs:LED_WS2812B-PLCC4" H 4650 3300 50  0001 L CNN
+F 2 "lib:LED_WS2812B-PLCC4" H 4650 3300 50  0001 L CNN
 F 3 "" H 4550 3250 60  0000 C CNN
 	1    4800 3300
@@
 F 0 "D303" H 5910 3580 50  0000 L CNN
 F 1 "WS2812B" H 6100 3300 50  0000 L CNN
-F 2 "LEDs:LED_WS2812B-PLCC4" H 6100 3300 50  0001 L CNN
+F 2 "lib:LED_WS2812B-PLCC4" H 6100 3300 50  0001 L CNN
 F 3 "" H 6000 3250 60  0000 C CNN
 	1    6250 3300
@@
 F 0 "D304" H 7360 3580 50  0000 L CNN
 F 1 "WS2812B" H 7550 3300 50  0000 L CNN
-F 2 "LEDs:LED_WS2812B-PLCC4" H 7550 3300 50  0001 L CNN
+F 2 "lib:LED_WS2812B-PLCC4" H 7550 3300 50  0001 L CNN
 F 3 "" H 7450 3250 60  0000 C CNN
 	1    7700 3300
@@
 F 0 "D305" H 3010 5180 50  0000 L CNN
 F 1 "WS2812B" H 3200 4900 50  0000 L CNN
-F 2 "LEDs:LED_WS2812B-PLCC4" H 3200 4900 50  0001 L CNN
+F 2 "lib:LED_WS2812B-PLCC4" H 3200 4900 50  0001 L CNN
 F 3 "" H 3100 4850 60  0000 C CNN
 	1    3350 4900
@@
 F 0 "D306" H 4460 5180 50  0000 L CNN
 F 1 "WS2812B" H 4650 4900 50  0000 L CNN
-F 2 "LEDs:LED_WS2812B-PLCC4" H 4650 4900 50  0001 L CNN
+F 2 "lib:LED_WS2812B-PLCC4" H 4650 4900 50  0001 L CNN
 F 3 "" H 4550 4850 60  0000 C CNN
 	1    4800 4900
@@
 F 0 "D307" H 5910 5180 50  0000 L CNN
 F 1 "WS2812B" H 6100 4900 50  0000 L CNN
-F 2 "LEDs:LED_WS2812B-PLCC4" H 6100 4900 50  0001 L CNN
+F 2 "lib:LED_WS2812B-PLCC4" H 6100 4900 50  0001 L CNN
 F 3 "" H 6000 4850 60  0000 C CNN
 	1    6250 4900
@@
 F 0 "D308" H 7360 5180 50  0000 L CNN
 F 1 "WS2812B" H 7550 4900 50  0000 L CNN
-F 2 "LEDs:LED_WS2812B-PLCC4" H 7550 4900 50  0001 L CNN
+F 2 "lib:LED_WS2812B-PLCC4" H 7550 4900 50  0001 L CNN
 F 3 "" H 7450 4850 60  0000 C CNN
 	1    7700 4900
