File: hardware/Power.sch (KiCad schematic (older format))
At the start: 5 parts

Commit message: Add annotations
Parts:
- gave numbers to parts that had none: 5
Changed lines of the file:
@@
 VUSB
 $Comp
-L MCP73831 U?
+L MCP73831 U201
 U 1 1 5779CF87
 P 5100 3500
-F 0 "U?" H 4900 3700 60  0000 C CNN
+F 0 "U201" H 4900 3700 60  0000 C CNN
 F 1 "MCP73831" H 5100 3300 60  0000 C CNN
 F 2 "" H 5100 3500 60  0000 C CNN
@@
 	5700 3600 5700 4050
 $Comp
-L GND #PWR?
+L GND #PWR201
 U 1 1 5779CFD2
 P 5700 4050
-F 0 "#PWR?" H 5700 3800 50  0001 C CNN
+F 0 "#PWR201" H 5700 3800 50  0001 C CNN
 F 1 "GND" H 5700 3900 50  0000 C CNN
 F 2 "" H 5700 4050 50  0000 C CNN
@@
 $EndComp
 $Comp
-L C C?
+L C C201
 U 1 1 5779D02A
 P 4300 3650
-F 0 "C?" H 4325 3750 50  0000 L CNN
+F 0 "C201" H 4325 3750 50  0000 L CNN
 F 1 "4.7uF" H 4325 3550 50  0000 L CNN
 F 2 "" H 4338 3500 50  0000 C CNN
@@
 	4300 3900 6500 3900
 $Comp
-L R R?
+L R R201
 U 1 1 5779D0FC
 P 5900 3700
-F 0 "R?" V 5980 3700 50  0000 C CNN
+F 0 "R201" V 5980 3700 50  0000 C CNN
 F 1 "2.0k" V 5900 3700 50  0000 C CNN
 F 2 "" V 5830 3700 50  0000 C CNN
@@
 Connection ~ 5700 3900
 $Comp
-L C C?
+L C C202
 U 1 1 5779D16F
 P 6150 3650
-F 0 "C?" H 6175 3750 50  0000 L CNN
+F 0 "C202" H 6175 3750 50  0000 L CNN
 F 1 "4.7uF" H 6175 3550 50  0000 L CNN
 F 2 "" H 6188 3500 50  0000 C CNN
@@
 	6150 3400 6150 3500
 $Comp
-L CONN_01X02 P?
+L CONN_01X02 P201
 U 1 1 5779D232
 P 6700 3650
-F 0 "P?" H 6700 3800 50  0000 C CNN
+F 0 "P201" H 6700 3800 50  0000 C CNN
 F 1 "CONN_01X02" V 6800 3650 50  0000 C CNN
 F 2 "" H 6700 3650 50  0000 C CNN

Commit message: Update footprints
Parts:
- C201, C202: footprint (none) -> Capacitors_SMD:C_0603
- R201: footprint (none) -> Resistors_SMD:R_0603
Changed lines of the file:
@@
 F 0 "U201" H 4900 3700 60  0000 C CNN
 F 1 "MCP73831" H 5100 3300 60  0000 C CNN
-F 2 "" H 5100 3500 60  0000 C CNN
+F 2 "" H 5100 3500 60  0001 C CNN
 F 3 "" H 5100 3500 60  0000 C CNN
 	1    5100 3500
@@
 	5700 3600 5700 4050
 $Comp
-L GND #PWR201
+L GND #PWR013
 U 1 1 5779CFD2
 P 5700 4050
-F 0 "#PWR201" H 5700 3800 50  0001 C CNN
+F 0 "#PWR013" H 5700 3800 50  0001 C CNN
 F 1 "GND" H 5700 3900 50  0000 C CNN
 F 2 "" H 5700 4050 50  0000 C CNN
@@
 F 0 "C201" H 4325 3750 50  0000 L CNN
 F 1 "4.7uF" H 4325 3550 50  0000 L CNN
-F 2 "" H 4338 3500 50  0000 C CNN
+F 2 "Capacitors_SMD:C_0603" H 4338 3500 50  0001 C CNN
 F 3 "" H 4300 3650 50  0000 C CNN
 	1    4300 3650
@@
 F 0 "R201" V 5980 3700 50  0000 C CNN
 F 1 "2.0k" V 5900 3700 50  0000 C CNN
-F 2 "" V 5830 3700 50  0000 C CNN
+F 2 "Resistors_SMD:R_0603" V 5830 3700 50  0001 C CNN
 F 3 "" H 5900 3700 50  0000 C CNN
 	1    5900 3700
@@
 F 0 "C202" H 6175 3750 50  0000 L CNN
 F 1 "4.7uF" H 6175 3550 50  0000 L CNN
-F 2 "" H 6188 3500 50  0000 C CNN
+F 2 "Capacitors_SMD:C_0603" H 6188 3500 50  0001 C CNN
 F 3 "" H 6150 3650 50  0000 C CNN
 	1    6150 3650
@@
 F 0 "P201" H 6700 3800 50  0000 C CNN
 F 1 "CONN_01X02" V 6800 3650 50  0000 C CNN
-F 2 "" H 6700 3650 50  0000 C CNN
+F 2 "" H 6700 3650 50  0001 C CNN
 F 3 "" H 6700 3650 50  0000 C CNN
 	1    6700 3650

Commit message: Update some footprint assignments
Parts:
- U201: footprint (none) -> TO_SOT_Packages_SMD:SOT-23-5
Changed lines of the file:
@@
 F 0 "U201" H 4900 3700 60  0000 C CNN
 F 1 "MCP73831" H 5100 3300 60  0000 C CNN
-F 2 "" H 5100 3500 60  0001 C CNN
+F 2 "TO_SOT_Packages_SMD:SOT-23-5" H 5100 3500 60  0001 C CNN
 F 3 "" H 5100 3500 60  0000 C CNN
 	1    5100 3500

Commit message: Update some footprint assignments
Parts:
- P201: footprint (none) -> lib:JST2
Changed lines of the file:
@@
 F 0 "P201" H 6700 3800 50  0000 C CNN
 F 1 "CONN_01X02" V 6800 3650 50  0000 C CNN
-F 2 "" H 6700 3650 50  0001 C CNN
+F 2 "lib:JST2" H 6700 3650 50  0001 C CNN
 F 3 "" H 6700 3650 50  0000 C CNN
 	1    6700 3650
