File: hardware/Power.sch (KiCad schematic (older format))
At the start: 5 parts, among them P201 CONN_01X02, U201 MCP73831

Commit message: Fix PMOS pinout
Parts:
- P201: footprint lib:JST2 -> lib:JST_PH_SMD
Changed lines of the file:
@@
 F 0 "P201" H 6700 3800 50  0000 C CNN
 F 1 "CONN_01X02" V 6800 3650 50  0000 C CNN
-F 2 "lib:JST2" H 6700 3650 50  0001 C CNN
+F 2 "lib:JST_PH_SMD" H 6700 3650 50  0001 C CNN
 F 3 "" H 6700 3650 50  0000 C CNN
 	1    6700 3650
